File: Kretsdiagram/Kretsdiagram/Kretsdiagram.kicad_sch (KiCad schematic)
At the start: 0 parts

Commit message: Ferdig
Parts:
- added A2: Arduino_UNO_R3, Module:Arduino_UNO_R3, symbol MCU_Module:Arduino_UNO_R3
- added BZ1: Buzzer, symbol Device:Buzzer
- added D1, D2, D3, D4, D5: LED, symbol Device:LED
- added LCD-I2C: ~, symbol New_Library:LCD-I2C
- added SW1, SW2, SW3: SW_Push, symbol Switch:SW_Push
Connections:
- new net: A2.13 (SDA/A4), LCD-I2C.3 (SDA)
- new net: A2.14 (SCL/A5), LCD-I2C.4 (SCL)
- new net: A2.20 (D5), SW1.1
- new net: A2.24 (D9), BZ1.1 (+)
- new net: A2.25 (D10), SW3.1
- new net: A2.27 (D12), SW2.1
- new net +5V: A2.5 (+5V), LCD-I2C.2 (VCC), SW1.2, SW2.2, SW3.2
- new net GND: A2.7 (GND), BZ1.2 (-), D1.1 (K), D2.1 (K), D3.1 (K), D4.1 (K), D5.1 (K), LCD-I2C.1 (GND)
